File: INPUT.kicad_sch (KiCad schematic)
At the start: 41 parts, among them J3 S7B-PH-K-S(LF)(SN), J4 S7B-PH-K-S(LF)(SN), P1 S7B-PH-SM4-TB(LF)(SN), P2 S7B-PH-SM4-TB(LF)(SN), U2 74HC240

Commit message: rev2 sent to fab
Added CHR RAM.
Changed board to 4 layers (was 2 layers).
Changed passives to 0603 (was 0402)
Fixed CIRAM-A10 not being hooked up
Fixed PPU-A10..A12 being hooked to VRAM but should have been.
Added more silkscreen for easier debugging.
Added filter inductor to 5V from USB-C.
Changed video out to stock (was THS7374)
Changed audio circuit to stock (was headphone amp IC)
Parts:
- C10, C11, C22, C23, C24, C29, C31, C7, C8: footprint Capacitor_SMD:C_0402_1005Metric -> Capacitor_SMD:C_0603_1608Metric_Pad1.08x0.95mm_HandSolder; Digikey 1292-1308-1-ND -> (none); MPN 0402N331J500CT -> (none)
- C50: footprint Capacitor_SMD:C_0402_1005Metric -> Capacitor_SMD:C_0603_1608Metric_Pad1.08x0.95mm_HandSolder; Digikey 1276-1509-2-ND -> (none); MPN CL05B104KO5NNWC -> (none); QOH 10000 -> (none)
- D1, D10, D11, D2, D5, D6, D7, D8, D9: footprint Package_TO_SOT_SMD:SOT-23 -> Package_TO_SOT_SMD:SOT-23_Handsoldering
- R11, R12, R14, R17, R18, R8: footprint Resistor_SMD:R_0402_1005Metric -> Resistor_SMD:R_0603_1608Metric_Pad0.98x0.95mm_HandSolder; Digikey P10.0KLCT-ND -> (none); MPN ERJ-2RKF1002X -> (none); QOH 5000 -> (none)
- R13, R28, R5: footprint Resistor_SMD:R_0402_1005Metric -> Resistor_SMD:R_0603_1608Metric_Pad0.98x0.95mm_HandSolder; Digikey 311-6.80KLRCT-ND -> (none); MPN RC0402FR-076K8L -> (none)

Commit message: filled out BOM
Parts:
- C10, C11, C22, C23, C24, C29, C31, C7, C8: Digikey (none) -> 399-C0603C331J5GAC7867CT-ND; MPN (none) -> C0603C331J5GAC7867
- C50: Digikey (none) -> 1276-CL10B104KB8WPNDCT-ND; MPN (none) -> CL10B104KB8WPND
- R11, R12, R14, R17, R18, R8: Digikey (none) -> RMCF0603FT10K0CT-ND; MPN (none) -> RMCF0603FT10K0
- R13, R28, R5: Digikey (none) -> 311-6.80KHRCT-ND; MPN (none) -> RMCF0603FT110RCT-ND
